File: kicad-project/c64-psu.sch (KiCad schematic (older format))
At the start: 49 parts, among them J1 Conn_01x01, J2 Conn_01x01, J3 Conn_01x01, J4 Conn_01x01, J5 Conn_01x01, J6 Conn_01x01, Q1 N-MOS, U1 LMR33630A, U2 MAX6399

Commit message: fixed bug: copper fill under spade connectors to prevent ground plane shorts
gerbers + bom redone
Parts:
- J1, J2, J3, J4, J5, J6: Mfr (none) -> Keystone; MfrCode (none) -> 1212-ST; MouserCode (none) -> 534-1212-ST
Changed lines of the file:
@@
 F 1 "Net-Tie_2" V 7200 4650 50  0000 C CNN
 F 2 "NetTie:NetTie-2_THT_Pad1.0mm" H 7200 4300 50  0001 C CNN
-F 3 "~" H 7200 4300 50  0001 C CNN
+F 3 "" H 7200 4300 50  0001 C CNN
 	1    7200 4300
 	1    0    0    -1
@@
 F 1 "TestPoint_2Pole" V 10145 3808 50  0000 L CNN
 F 2 "TestPoint:TestPoint_2Pads_Pitch2.54mm_Drill0.8mm" H 10100 3750 50  0001 C CNN
-F 3 "~" H 10100 3750 50  0001 C CNN
+F 3 "" H 10100 3750 50  0001 C CNN
 	1    10100 3750
 	0    1    1    0
@@
 F 1 "TestPoint_2Pole" V 10095 1458 50  0000 L CNN
 F 2 "TestPoint:TestPoint_2Pads_Pitch2.54mm_Drill0.8mm" H 10050 1400 50  0001 C CNN
-F 3 "~" H 10050 1400 50  0001 C CNN
+F 3 "" H 10050 1400 50  0001 C CNN
 	1    10050 1400
 	0    1    1    0
@@
 F 1 "TestPoint_2Pole" H 3550 3700 50  0000 L CNN
 F 2 "TestPoint:TestPoint_2Pads_Pitch2.54mm_Drill0.8mm" H 3400 3650 50  0001 C CNN
-F 3 "~" H 3400 3650 50  0001 C CNN
+F 3 "" H 3400 3650 50  0001 C CNN
 	1    3400 3650
 	0    1    1    0
@@
 F 1 "Conn_01x01" H 10580 2951 50  0000 L CNN
 F 2 "c64-psu:spade_4.8mm" H 10500 3000 50  0001 C CNN
-F 3 "~" H 10500 3000 50  0001 C CNN
+F 3 "" H 10500 3000 50  0001 C CNN
+F 4 "Keystone" H 0   0   50  0001 C CNN "Mfr"
+F 5 "1212-ST" H 0   0   50  0001 C CNN "MfrCode"
+F 6 "534-1212-ST" H 0   0   50  0001 C CNN "MouserCode"
 	1    10500 3000
 	1    0    0    -1
@@
 F 1 "Conn_01x01" H 10580 4251 50  0000 L CNN
 F 2 "c64-psu:spade_4.8mm" H 10500 4300 50  0001 C CNN
-F 3 "~" H 10500 4300 50  0001 C CNN
+F 3 "" H 10500 4300 50  0001 C CNN
+F 4 "Keystone" H 0   0   50  0001 C CNN "Mfr"
+F 5 "1212-ST" H 0   0   50  0001 C CNN "MfrCode"
+F 6 "534-1212-ST" H 0   0   50  0001 C CNN "MouserCode"
 	1    10500 4300
 	1    0    0    -1
@@
 F 1 "Conn_01x01" H 10580 1651 50  0000 L CNN
 F 2 "c64-psu:spade_4.8mm" H 10500 1700 50  0001 C CNN
-F 3 "~" H 10500 1700 50  0001 C CNN
+F 3 "" H 10500 1700 50  0001 C CNN
+F 4 "Keystone" H 0   0   50  0001 C CNN "Mfr"
+F 5 "1212-ST" H 0   0   50  0001 C CNN "MfrCode"
+F 6 "534-1212-ST" H 0   0   50  0001 C CNN "MouserCode"
 	1    10500 1700
 	1    0    0    -1
@@
 F 1 "Conn_01x01" H 10580 1051 50  0000 L CNN
 F 2 "c64-psu:spade_4.8mm" H 10500 1100 50  0001 C CNN
-F 3 "~" H 10500 1100 50  0001 C CNN
+F 3 "" H 10500 1100 50  0001 C CNN
+F 4 "Keystone" H 0   0   50  0001 C CNN "Mfr"
+F 5 "1212-ST" H 0   0   50  0001 C CNN "MfrCode"
+F 6 "534-1212-ST" H 0   0   50  0001 C CNN "MouserCode"
 	1    10500 1100
 	1    0    0    -1
@@
 F 1 "Conn_01x01" H 1070 966 50  0000 C CNN
 F 2 "c64-psu:spade_4.8mm" H 1150 1100 50  0001 C CNN
-F 3 "~" H 1150 1100 50  0001 C CNN
+F 3 "" H 1150 1100 50  0001 C CNN
+F 4 "Keystone" H 0   0   50  0001 C CNN "Mfr"
+F 5 "1212-ST" H 0   0   50  0001 C CNN "MfrCode"
+F 6 "534-1212-ST" H 0   0   50  0001 C CNN "MouserCode"
 	1    1150 1100
 	-1   0    0    1
@@
 F 1 "Conn_01x01" H 1070 1466 50  0000 C CNN
 F 2 "c64-psu:spade_4.8mm" H 1150 1600 50  0001 C CNN
-F 3 "~" H 1150 1600 50  0001 C CNN
+F 3 "" H 1150 1600 50  0001 C CNN
+F 4 "Keystone" H 0   0   50  0001 C CNN "Mfr"
+F 5 "1212-ST" H 0   0   50  0001 C CNN "MfrCode"
+F 6 "534-1212-ST" H 0   0   50  0001 C CNN "MouserCode"
 	1    1150 1600
 	-1   0    0    1
